File: Electronics/rev2/paperd.ink_main_pcb.kicad_pcb (KiCad board)
At the start: 4 copper layers, 92.1 x 78.1 mm, 84 parts, among them J1 USB_B_Micro, J3 Conn_01x14, J4 EXT_CONN, Q1 DMP2035, Q2 T2N7002BK, Q3 DMP2035, Q4 DMP2035, Q5 DMP2035, Q6 UMH3N, Q7 UMH3N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

Commit message: split PCB into main and front
Routing:
- net ~FPC_LED_R: track 22.1 -> 9.81 mm
- net ~FPC_LED_B: track 21.8 -> 13.8 mm
Changed lines of the file:
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@@
   (general
     (thickness 0.8)
-    (drawings 26)
-    (tracks 1612)
+    (drawings 25)
+    (tracks 1604)
     (modules 84)
     (nets 110)
@@
   (paper "A4")
   (layers
-    (0 "F.Cu" signal hide)
+    (0 "F.Cu" signal)
     (1 "In1.Cu" mixed hide)
     (2 "In2.Cu" power hide)
@@
     (visible_elements FFFDFF7F)
     (pcbplotparams
-      (layerselection 0x010fc_ffffffff)
+      (layerselection 0x310fc_ffffffff)
       (usegerberextensions true)
       (usegerberattributes false)
@@
       (drillshape 0)
       (scaleselection 1)
-      (outputdirectory "Output/Gerbers/")
+      (outputdirectory "Output/Gerbers_Main_PCB/")
     )
   )
@@
     (pad "1" smd roundrect (at -1.9375 1.25 90) (size 0.825 0.25) (layers "B.Cu" "B.Paste" "B.Mask") (roundrect_rratio 0.25)
       (net 107 "Net-(U4-Pad1)"))
-    (pad "" smd roundrect (at 0.65 -0.65 90) (size 1.05 1.05) (layers "B.Paste") (roundrect_rratio 0.238095))
-    (pad "" smd roundrect (at 0.65 0.65 90) (size 1.05 1.05) (layers "B.Paste") (roundrect_rratio 0.238095))
-    (pad "" smd roundrect (at -0.65 -0.65 90) (size 1.05 1.05) (layers "B.Paste") (roundrect_rratio 0.238095))
-    (pad "" smd roundrect (at -0.65 0.65 90) (size 1.05 1.05) (layers "B.Paste") (roundrect_rratio 0.238095))
-    (pad "25" smd roundrect (at 0 0 90) (size 2.6 2.6) (layers "B.Cu" "B.Mask") (roundrect_rratio 0.096154)
+    (pad "" smd roundrect (at 0.65 -0.65 90) (size 1.05 1.05) (layers "B.Paste") (roundrect_rratio 0.2380942857142857))
+    (pad "" smd roundrect (at 0.65 0.65 90) (size 1.05 1.05) (layers "B.Paste") (roundrect_rratio 0.2380942857142857))
+    (pad "" smd roundrect (at -0.65 -0.65 90) (size 1.05 1.05) (layers "B.Paste") (roundrect_rratio 0.2380942857142857))
+    (pad "" smd roundrect (at -0.65 0.65 90) (size 1.05 1.05) (layers "B.Paste") (roundrect_rratio 0.2380942857142857))
+    (pad "25" smd roundrect (at 0 0 90) (size 2.6 2.6) (layers "B.Cu" "B.Mask") (roundrect_rratio 0.09615384615384616)
       (net 1 "GND"))
     (model "${KISYS3DMOD}/Package_DFN_QFN.3dshapes/QFN-24-1EP_4x4mm_P0.5mm_EP2.6x2.6mm.wrl"
@@
     (effects (font (size 0.8128 1) (thickness 0.1524)) (justify mirror))
   )
-  (gr_line (start 189.55 140.01) (end 194.55 140.04) (layer "Eco1.User") (width 0.15))
   (gr_line (start 104.256 113.854) (end 104.002 113.346) (layer "B.SilkS") (width 0.1524))
   (gr_line (start 104.764 113.6) (end 104.256 113.854) (layer "B.SilkS") (width 0.1524))
@@
   (segment (start 182.05 134.11) (end 181.87 134.29) (width 0.1016) (layer "F.Cu") (net 74))
   (segment (start 185.06 134.06) (end 185.01 134.11) (width 0.1016) (layer "F.Cu") (net 74) (status 30))
-  (segment (start 193.06 139.11) (end 193.06 140.28) (width 0.1016) (layer "F.Cu") (net 74))
-  (segment (start 188.01 134.06) (end 193.06 139.11) (width 0.1016) (layer "F.Cu") (net 74))
-  (segment (start 185.06 134.06) (end 188.01 134.06) (width 0.1016) (layer "F.Cu") (net 74) (status 10))
-  (segment (start 192.56 140.28) (end 193.56 140.28) (width 0.1016) (layer "F.Cu") (net 74))
   (segment (start 183.34 129.415) (end 183.34 136.73) (width 0.1016) (layer "B.Cu") (net 75) (status 10))
   (segment (start 185.06 138.56) (end 185.06 138.06) (width 0.1016) (layer "F.Cu") (net 75) (status 30))
-  (segment (start 191.06 139.71) (end 191.06 140.28) (width 0.1016) (layer "F.Cu") (net 75))
-  (segment (start 189.91 138.56) (end 191.06 139.71) (width 0.1016) (layer "F.Cu") (net 75))
-  (segment (start 185.06 138.56) (end 189.91 138.56) (width 0.1016) (layer "F.Cu") (net 75) (status 10))
-  (segment (start 191.06 140.28) (end 192.06 140.28) (width 0.1016) (layer "F.Cu") (net 75))
   (segment (start 184.96 136.16) (end 185.06 136.06) (width 0.1016) (layer "F.Cu") (net 76) (status 30))
   (via (at 189.89 70.76) (size 0.45) (drill 0.2) (layers "F.Cu" "B.Cu") (net 4))
